File: Kicad/Untitled/Untitled.kicad_sch (KiCad schematic)
At the start: 10 parts, among them J1 Conn_01x16_Pin, P1 USB_C_Plug_USB2.0, U1 NCP1117-3.3_TO252, U2 ESP32-S3, Y1 ABM8-40.000MHZ-B2-T

Commit message: update schematic, more info in journakl
Parts:
- removed P1: USB_C_Plug_USB2.0, symbol Connector:USB_C_Plug_USB2.0
- removed Y1: ABM8-40.000MHZ-B2-T, ABM8-40.000MHZ-B2-T:XTAL_ABM8-40.000MHZ-B2-T, symbol ABM8-40.000MHZ-B2-T:ABM8-40.000MHZ-B2-T
- added J2: USB_C_Receptacle_USB2.0_14P, symbol Connector:USB_C_Receptacle_USB2.0_14P
- added R4: 5.1k, symbol Device:R
Connections:
- net BGPIO1: now also J1.1 (Pin_1)
- net BGPIO2: now also J1.2 (Pin_2)
- net BGPIO3: now also J1.3 (Pin_3)
- net GND: now also J2.A1 (GND), J2.A12 (GND), J2.B1 (GND), J2.B12 (GND), J2.S1 (SHIELD), R4.2
- net USBD+: now also J2.A6 (D+), J2.B6 (D+)
- net USBD-: now also J2.A7 (D-), J2.B7 (D-)
- net VBUS: now also J2.A4 (VBUS), J2.A9 (VBUS), J2.B4 (VBUS), J2.B9 (VBUS)
- net at R1.1: now also J2.B5 (CC2)
- net BGPIO4: now reaches J1.4 (Pin_4)
- net BGPIO4: now also U2.18 (GPIO13)
- new net: J2.A5 (CC1), R4.1
Other:
- note removed: "Clock"
- moved on the sheet: J1, R1, R2, R3, U2

Commit message: journal
Parts:
- added C3, C4: 6.8pF, symbol Device:C
- added J3: Conn_01x20_Pin, symbol Connector:Conn_01x20_Pin
- added J4: Conn_01x05_Pin, symbol Connector:Conn_01x05_Pin
- added R5: 1k, symbol Device:R
- added Y1: 40 MHz, symbol Device:Crystal_GND24
Connections:
- net GND: now also C3.1, C4.1, Y1.2, Y1.4
- net at U2.25 (GPIO19/USB_D-): now also R3.1
- net at U2.27 (GPIO21): no longer R3.1
- net XIN: now reaches U2.53 (XTAL_N)
- net XIN: now also C3.2, Y1.3
- net XOUT: now reaches U2.54 (XTAL_P)
- net XOUT: now also R5.2
- new net: C4.2, R5.1, Y1.1
Other:
- moved on the sheet: R3

Commit message: journal entry explains
Parts:
- removed J4: Conn_01x05_Pin, symbol Connector:Conn_01x05_Pin
- added C10, C11, C12, C13, C14: 0.1uF, symbol Device:C
- added C15: 1uF, symbol Device:C
- added C5, C6: 12pF, symbol Device:C
- added C7, C8: 10uF, symbol Device:C
- added J4: Conn_01x04_Socket, symbol Connector:Conn_01x04_Socket
- added J6: Screw_Terminal_01x02, symbol Connector:Screw_Terminal_01x02
- added R6: 10k, symbol Device:R
- added R7: 200, symbol Device:R
- added SW1, SW2: SW_Push_45deg, symbol Switch:SW_Push_45deg
- added SW3, SW4: SW_Push, symbol Switch:SW_Push
- added U3: NCP1117-3.3_TO252, Package_TO_SOT_SMD:TO-252-2, symbol Regulator_Linear:NCP1117-3.3_TO252
- added Y2: 32.768kHz, symbol Device:Crystal
- C3, C4: value 6.8pF -> 12pF
Connections:
- net +3V3: now also J1.14 (Pin_14), C10.1, C11.1, C12.1, C13.1, C14.1, C15.1, C7.1, R6.2, U3.2 (VO)
- net BGPIO1: now also J1.13 (Pin_13)
- net BGPIO2: now also J1.12 (Pin_12)
- net BGPIO3: now also J1.11 (Pin_11)
- net BGPIO4: now also J3.4 (Pin_4)
- net GND: now also J1.16 (Pin_16), J3.20 (Pin_20), C10.2, C11.2, C12.2, C13.2, C14.2, C15.2, C5.2, C6.2, C7.2, C8.2, J4.4 (Pin_4), J6.2 (Pin_2), SW1.1, SW2.2, SW3.2, SW4.2, U3.1 (GND)
- net VBUS: now also J1.15 (Pin_15), C8.1, J6.1 (Pin_1), U3.3 (VI)
- net BGPIO8: now reaches J1.10 (Pin_10)
- net BGPIO8: now also U2.9 (GPIO4)
- net SCL: now reaches J1.5 (Pin_5)
- net SCL: now also U2.13 (GPIO8)
- net SDA: now reaches J1.6 (Pin_6)
- net SDA: now also U2.14 (GPIO9)
- net BGPIO11: now reaches J1.7 (Pin_7)
- net BGPIO11: now also U2.12 (GPIO7)
- net BGPIO10: now reaches J1.8 (Pin_8)
- net BGPIO10: now also U2.11 (GPIO6)
- net BGPIO9: now reaches J1.9 (Pin_9)
- net BGPIO9: now also U2.10 (GPIO5)
- net BGPIO7: now reaches J3.1 (Pin_1)
- net BGPIO7: now also U2.24 (GPIO18)
- net BGPIO6: now reaches J3.2 (Pin_2)
- net BGPIO6: now also U2.23 (GPIO17)
- net BGPIO5: now reaches J3.3 (Pin_3)
- net BGPIO5: now also U2.19 (GPIO14)
- net BGPIO12: now reaches J3.5 (Pin_5)
- net BGPIO12: now also U2.27 (GPIO21)
- net XTAL_32K_P: now reaches U2.21 (XTAL_32K_P)
- net XTAL_32K_P: now also R7.2
- net XTAL_32K_N: now reaches U2.22 (XTAL_32K_N)
- net XTAL_32K_N: now also C5.1, Y2.1
- net at U2.4 (CHIP_PU): now also R6.1, SW2.1
- net RXD: now reaches U2.49 (U0TXD)
- net RXD: now also J4.2 (Pin_2)
- net at U2.5 (GPIO0): now also SW1.2
- net TXD: now reaches U2.50 (U0RXD)
- net TXD: now also J4.3 (Pin_3)
- net at U2.51 (GPIO45): now also SW3.1
- net at U2.52 (GPIO46): now also SW4.1
- new net: C6.1, R7.1, Y2.2
- new net +3.3V: J4.1 (Pin_1)
- no-connect marks 0 -> 1
Other:
- note added: "3V3 & GND Pin Breakouts"
- note added: "ESP32 Devboard Schematic - Wiring"
- note added: "GPIO PIN Breakouts"
- note added: "Lithium ion battery screw terminal"
- note added: "USB-UART FOR FIRST TIME FLASHING, ALSO FOR ANY CRITICAL CHANGES IN CASE EVERYTHING ELSE FAILS"
- moved on the sheet: C1, C2, C3, C4, J1, J2, J3, R1, R2, R3, R4, R5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

Commit message: journal update
Parts:
- added C16, C18: 1uF, symbol Device:C
- added C17, C9: 0.1uF, symbol Device:C
- added D1: LED, symbol Device:LED
- added L1: 2nH, symbol Device:L
- added R10, R11, R12, R13, R14: 0, symbol Device:R
- added R8: 10k, symbol Device:R
- added R9: 440, symbol Device:R
- added U4: APS6404L-3SQRx-ZR, Package_SON:Winbond_USON-8-1EP_3x2mm_P0.5mm_EP0.2x1.6mm, symbol Memory_RAM:APS6404L-3SQRx-ZR
- C13: value 0.1uF -> 1uF
- C14: value 0.1uF -> 10uF
- C15: value 1uF -> 10nF
Connections:
- net +3V3: now also C12.2, C13.2, C14.2, J3.18 (Pin_18), U2.20 (VDD3P3_RTC), U2.46 (VDD3P3_CPU), U2.55 (VDDA), U2.56 (VDDA), C16.1, C9.1, D1.2 (A), L1.1, R8.2; no longer C11.1, C12.1, C13.1, C14.1
- net BGPIO1: no longer J1.13 (Pin_13)
- net BGPIO10: now also J1.12 (Pin_12); no longer J1.8 (Pin_8)
- net BGPIO11: now also J1.13 (Pin_13); no longer J1.7 (Pin_7)
- net BGPIO12: now also J3.1 (Pin_1); no longer J3.5 (Pin_5)
- net BGPIO2: no longer J1.12 (Pin_12)
- net BGPIO3: no longer J1.11 (Pin_11)
- net BGPIO4: no longer J3.4 (Pin_4)
- net BGPIO5: now also J1.5 (Pin_5); no longer J3.3 (Pin_3)
- net BGPIO6: now also J1.6 (Pin_6); no longer J3.2 (Pin_2)
- net BGPIO7: now also J1.7 (Pin_7); no longer J3.1 (Pin_1)
- net BGPIO8: now also J1.8 (Pin_8); no longer J1.10 (Pin_10)
- net GND: now also C11.1, C12.1, C13.1, C14.1, C16.2, C17.2, C18.2, C9.2, R9.2, U4.4 (VSS), U4.9 (EPAD); no longer C11.2, C12.2, C13.2, C14.2
- net SCL: now also J1.10 (Pin_10); no longer J1.5 (Pin_5)
- net SDA: now also J1.11 (Pin_11); no longer J1.6 (Pin_6)
- net VBUS: now also J3.19 (Pin_19)
- net at SW1.2, U2.5 (GPIO0): now also R8.1
- net at U2.2 (VDD3P3), U2.3 (VDD3P3): now also C11.2, L1.2
- net VDD_SPI: now reaches U2.29 (VDD_SPI)
- net VDD_SPI: now also C17.1, C18.1, U4.8 (VDD)
- net at U2.30 (SPIHD): now also R13.1
- net at U2.31 (SPIWP): now also R14.1
- net at U2.33 (SPICLK): now also R12.1
- net at U2.34 (SPIQ): now also R10.1
- net at U2.35 (SPID): now also R11.1
- net CHIPSELECT: now reaches U2.39 (GPIO34)
- net CHIPSELECT: now also U4.1 (~{CE})
- new net: D1.1 (K), R9.1
- new net SPICLK: R12.2, U4.6 (SCLK)
- new net SPID: R11.2, U4.5 (SI/SIO0)
- new net SPIHD: R13.2, U4.7 (SIO3)
- new net SPIQ: R10.2, U4.2 (SO/SIO1)
- new net SPIWP: R14.2, U4.3 (SIO2)
- no-connect marks 1 -> 3
Other:
- note added: "CRYSTAL SETUP"
- note added: "PSRAM"
- note added: "Status LED"
- note added: "USB-C"
- moved on the sheet: R2, R3, R5, R6, R7, SW1, SW2, SW3, SW4, U2, Y1

Commit message: journal update
Parts:
- removed J3: Conn_01x20_Pin, symbol Connector:Conn_01x20_Pin
- added C10: 10uF, Capacitor_SMD:C_0201_0603Metric, symbol Device:C
- added C9: 1uF, Capacitor_SMD:C_0402_1005Metric, symbol Device:C
- added D2: D, Diode_SMD:D_0201_0603Metric, symbol Device:D
- added J5: Conn_01x04_Socket, Connector_PinSocket_2.54mm:PinSocket_1x04_P2.54mm_Horizontal, symbol Connector:Conn_01x04_Socket
- added J6: Conn_01x13_Pin, Connector_PinHeader_2.54mm:PinHeader_1x13_P2.54mm_Vertical, symbol Connector:Conn_01x13_Pin
- C1: renamed from C8; footprint (none) -> Capacitor_SMD:C_0201_0603Metric
- C11: renamed from C14; footprint (none) -> Capacitor_SMD:C_0201_0603Metric
- C12: renamed from C13; footprint (none) -> Capacitor_SMD:C_0402_1005Metric
- C13: renamed from C12; footprint (none) -> Capacitor_SMD:C_0402_1005Metric
- C14: renamed from C16; footprint (none) -> Capacitor_SMD:C_0402_1005Metric
- C15: renamed from C11; footprint (none) -> Capacitor_SMD:C_0402_1005Metric
- C16: renamed from C15; footprint (none) -> Capacitor_SMD:C_0402_1005Metric
- C17: renamed from C9; footprint (none) -> Capacitor_SMD:C_0402_1005Metric
- C18: renamed from C10; footprint (none) -> Capacitor_SMD:C_0402_1005Metric
- C19: renamed from C17; footprint (none) -> Capacitor_SMD:C_0402_1005Metric
- C2: renamed from C1; footprint (none) -> Capacitor_SMD:C_0201_0603Metric
- C20: renamed from C18; footprint (none) -> Capacitor_SMD:C_0402_1005Metric
- C3: renamed from C7; footprint (none) -> Capacitor_SMD:C_0201_0603Metric
- C4: renamed from C2; footprint (none) -> Capacitor_SMD:C_0201_0603Metric
- C5: renamed from C3; footprint (none) -> Capacitor_SMD:C_0402_1005Metric
- C6: renamed from C4; footprint (none) -> Capacitor_SMD:C_0402_1005Metric
- C7: renamed from C6; footprint (none) -> Capacitor_SMD:C_0402_1005Metric
- C8: renamed from C5; footprint (none) -> Capacitor_SMD:C_0402_1005Metric
- D1: footprint (none) -> LED_SMD:LED_WS2812B-Mini_PLCC4_3.5x3.5mm
- J1: renamed from J2; footprint (none) -> Connector_USB:USB_C_Receptacle_Amphenol_124019772112A
- J2: renamed from J4; footprint (none) -> Connector_PinSocket_2.54mm:PinSocket_1x04_P2.54mm_Horizontal
- J3: renamed from J6; footprint (none) -> TerminalBlock:TerminalBlock_Altech_AK300-2_P5.00mm
- J4: renamed from J1; footprint (none) -> Connector_PinHeader_2.54mm:PinHeader_1x16_P2.54mm_Vertical
- L1: footprint (none) -> Inductor_SMD:L_6.3x6.3_H3
- R1: renamed from R4; footprint (none) -> Resistor_SMD:R_0201_0603Metric
- R10: renamed from R14; footprint (none) -> Resistor_SMD:R_0201_0603Metric
- R11: renamed from R12; footprint (none) -> Resistor_SMD:R_0201_0603Metric
- R12: renamed from R10; footprint (none) -> Resistor_SMD:R_0201_0603Metric
- R13: renamed from R11; footprint (none) -> Resistor_SMD:R_0201_0603Metric
- R14: renamed from R6; footprint (none) -> Resistor_SMD:R_0201_0603Metric
- R2: renamed from R1; footprint (none) -> Resistor_SMD:R_0201_0603Metric
- R3: renamed from R9; footprint (none) -> Resistor_SMD:R_0201_0603Metric
- R4: renamed from R7; footprint (none) -> Resistor_SMD:R_0201_0603Metric
- R5: footprint (none) -> Resistor_SMD:R_0201_0603Metric
- R6: renamed from R8; footprint (none) -> Resistor_SMD:R_0201_0603Metric
- R7: renamed from R3; value 27 -> 22; footprint (none) -> Resistor_SMD:R_0201_0603Metric
- R8: renamed from R2; value 27 -> 22; footprint (none) -> Resistor_SMD:R_0201_0603Metric
- R9: renamed from R13; footprint (none) -> Resistor_SMD:R_0201_0603Metric
- SW1, SW2, SW3, SW4: footprint (none) -> Button_Switch_SMD:SW_Push_SPST_NO_Alps_SKRK
- Y1: renamed from Y2; footprint (none) -> AB38T_32_768KHZ:XTAL_AB38T-32.768KHZ
- Y2: renamed from Y1; footprint (none) -> CX2016DB40000D0FLJCC:OSC_CX2016DB40000D0FLJCC
- renumbered U3 to U1, U1 to U2, U4 to U3, U2 to U4
Connections:
- net +3.3V is gone; now on net +3V3: J2.1 (Pin_1)
- net VDD_SPI is gone; now on net +3V3: C19.1, C20.1, U3.8 (VDD), U4.29 (VDD_SPI)
- net +3V3: now also C10.1, C9.1, J6.11 (Pin_11)
- net GND: now also C10.2, C9.2, J6.13 (Pin_13)
- net VBUS: now also D2.2 (A), J6.12 (Pin_12); no longer C1.1, C2.1, J3.1 (Pin_1), U1.3 (VI), U2.3 (VI)
- net SPICS1: now reaches U4.28 (SPICS1)
- net SPICS1: now also U3.1 (~{CE})
- net IO16: now reaches U4.38 (GPIO33)
- net IO16: now also J6.5 (Pin_5)
- net IO18: now reaches U4.40 (GPIO35)
- net IO18: now also J6.7 (Pin_7)
- net IO19: now reaches U4.41 (GPIO36)
- net IO19: now also J6.8 (Pin_8)
- net IO20: now reaches U4.42 (GPIO37)
- net IO20: now also J6.9 (Pin_9)
- net IO21: now reaches U4.43 (GPIO38)
- net IO21: now also J6.10 (Pin_10)
- net MTCK: now reaches U4.44 (MTCK)
- net MTCK: now also J5.1 (Pin_1)
- net MTDO: now reaches U4.45 (MTDO)
- net MTDO: now also J5.2 (Pin_2)
- net MTDI: now reaches U4.47 (MTDI)
- net MTDI: now also J5.3 (Pin_3)
- net MTMS: now reaches U4.48 (MTMS)
- net MTMS: now also J5.4 (Pin_4)
- net IO1: now reaches U4.6 (GPIO1)
- net IO1: now also J4.1 (Pin_1)
- net IO2: now reaches U4.7 (GPIO2)
- net IO2: now also J4.2 (Pin_2)
- net IO3: now reaches U4.8 (GPIO3)
- net IO3: now also J4.3 (Pin_3)
- net BGPIO1 renamed IO8
- net IO8: now also J4.8 (Pin_8); no longer J4.1 (Pin_1)
- net BGPIO10 renamed IO10
- net IO10: now also U4.17 (GPIO12); no longer U4.11 (GPIO6)
- net BGPIO11 renamed IO11
- net IO11: now also U4.18 (GPIO13); no longer U4.12 (GPIO7)
- net BGPIO12 renamed IO15
- net IO15: now also J6.4 (Pin_4)
- net BGPIO2 renamed IO9
- net IO9: now also J4.9 (Pin_9); no longer J4.2 (Pin_2)
- removed net BGPIO3: J4.3 (Pin_3), U4.17 (GPIO12)
- net BGPIO4 renamed IO4
- net IO4: now also U4.9 (GPIO4); no longer U4.18 (GPIO13)
- net BGPIO5 renamed IO12
- net IO12: now also J6.1 (Pin_1); no longer J4.5 (Pin_5)
- net BGPIO6 renamed IO13
- net IO13: now also J6.2 (Pin_2); no longer J4.6 (Pin_6)
- net BGPIO7 renamed IO14
- net IO14: now also J6.3 (Pin_3); no longer J4.7 (Pin_7)
- removed net BGPIO8: J4.8 (Pin_8), U4.9 (GPIO4)
- net BGPIO9 renamed IO5
- net IO5: now also J4.5 (Pin_5); no longer J4.9 (Pin_9)
- net CHIPSELECT renamed IO17
- net IO17: now also J6.6 (Pin_6); no longer U3.1 (~{CE})
- new net: C2.1, D2.1 (K), U2.3 (VI)
- new net: C1.1, J3.1 (Pin_1), U1.3 (VI)
- new net IO6: J4.6 (Pin_6), U4.11 (GPIO6)
- new net IO7: J4.7 (Pin_7), U4.12 (GPIO7)
- no-connect marks 3 -> 4
Other:
- moved on the sheet: C11, C12, C13, C14, C15, C16, C17, C18, C19, C20, D1, J4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

Commit message: journal
Parts:
- removed D2: D, Diode_SMD:D_0201_0603Metric, symbol Device:D
- removed L1: 2nH, Inductor_SMD:L_6.3x6.3_H3, symbol Device:L
- added D2, D3: 1N4148WT, Diode_SMD:D_SOD-523, symbol Diode:1N4148WT
- J2, J5: footprint Connector_PinSocket_2.54mm:PinSocket_1x04_P2.54mm_Horizontal -> Connector_PinSocket_2.54mm:PinSocket_1x04_P2.54mm_Vertical
Connections:
- net +3V3: now also C15.2, U4.2 (VDD3P3), U4.3 (VDD3P3), D2.1 (K), D3.1 (K), D3.2 (A); no longer C4.1, U2.2 (VO)
- net VBUS: now also C2.1, U2.3 (VI)
- new net: C4.1, D2.2 (A), U2.2 (VO)
Changed lines of the file:
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@@
 	)
 	(junction
+		(at 76.2 109.22)
+		(diameter 0)
+		(color 0 0 0 0)
+	)
+	(junction
 		(at 212.09 52.07)
 		(diameter 0)
@@
 	(wire
 		(pts
+			(xy 77.47 109.22) (xy 76.2 109.22)
+		)
+		(stroke
+			(width 0)
+			(type default)
+		)
+	)
+	(wire
+		(pts
 			(xy 236.22 74.93) (xy 236.22 77.47)
 		)
@@
 	(wire
 		(pts
-			(xy 93.98 149.86) (xy 83.82 149.86)
+			(xy 93.98 149.86) (xy 92.71 149.86)
 		)
 		(stroke
@@
 	(wire
 		(pts
-			(xy 49.53 149.86) (xy 52.07 149.86)
+			(xy 49.53 149.86) (xy 66.04 149.86)
 		)
 		(stroke
@@
 	(wire
 		(pts
-			(xy 212.09 52.07) (xy 209.55 52.07)
-		)
-		(stroke
-			(width 0)
-			(type default)
-		)
-	)
-	(wire
-		(pts
 			(xy 140.97 72.39) (xy 147.32 72.39)
 		)
@@
 	(wire
 		(pts
+			(xy 85.09 149.86) (xy 83.82 149.86)
+		)
+		(stroke
+			(width 0)
+			(type default)
+		)
+	)
+	(wire
+		(pts
 			(xy 207.01 142.24) (xy 208.28 142.24)
 		)
@@
 	(wire
 		(pts
-			(xy 201.93 52.07) (xy 200.66 52.07)
+			(xy 200.66 52.07) (xy 212.09 52.07)
 		)
 		(stroke
@@
 	(wire
 		(pts
-			(xy 59.69 149.86) (xy 66.04 149.86)
-		)
-		(stroke
-			(width 0)
-			(type default)
-		)
-	)
-	(wire
-		(pts
 			(xy 280.67 144.78) (xy 274.32 144.78)
 		)
@@
 	)
 	(symbol
+		(lib_id "Diode:1N4148WT")
+		(at 88.9 149.86 180)
+		(unit 1)
+		(exclude_from_sim no)
+		(in_bom yes)
+		(on_board yes)
+		(dnp no)
+		(fields_autoplaced yes)
+		(property "Reference" "D2"
+			(at 88.9 143.51 0)
+			(effects
+				(font
+					(size 1.27 1.27)
+				)
+			)
+		)
+		(property "Value" "1N4148WT"
+			(at 88.9 146.05 0)
+			(effects
+				(font
+					(size 1.27 1.27)
+				)
+			)
+		)
+		(property "Footprint" "Diode_SMD:D_SOD-523"
+			(at 88.9 145.415 0)
+			(effects
+				(font
+					(size 1.27 1.27)
+				)
+				(hide yes)
+			)
+		)
+		(property "Datasheet" "https://www.diodes.com/assets/Datasheets/ds30396.pdf"
+			(at 88.9 149.86 0)
+			(effects
+				(font
+					(size 1.27 1.27)
+				)
+				(hide yes)
+			)
+		)
+		(property "Description" "75V 0.15A Fast switching Diode, SOD-523"
+			(at 88.9 149.86 0)
+			(effects
+				(font
+					(size 1.27 1.27)
+				)
+				(hide yes)
+			)
+		)
+		(property "Sim.Device" "D"
+			(at 88.9 149.86 0)
+			(effects
+				(font
+					(size 1.27 1.27)
+				)
+				(hide yes)
+			)
+		)
+		(property "Sim.Pins" "1=K 2=A"
+			(at 88.9 149.86 0)
+			(effects
+				(font
+					(size 1.27 1.27)
+				)
+				(hide yes)
+			)
+		)
+		(pin "2"
+		)
+		(pin "1"
+		)
+		(instances
+			(project ""
+				(path "/6663287f-38c5-4c19-8add-d68d3434afcd"
+					(reference "D2")
+					(unit 1)
+				)
+			)
+		)
+	)
+	(symbol
 		(lib_id "Connector:Conn_01x16_Pin")
 		(at 83.82 85.09 0)
@@
 	(symbol
 		(lib_id "power:+3V3")
-		(at 76.2 109.22 0)
+		(at 77.47 109.22 0)
 		(unit 1)
 		(exclude_from_sim no)
@@
 		(fields_autoplaced yes)
 		(property "Reference" "#PWR09"
-			(at 76.2 113.03 0)
+			(at 77.47 113.03 0)
 			(effects
 				(font
@@
 		)
 		(property "Value" "+3V3"
-			(at 76.2 104.14 0)
+			(at 77.47 104.14 0)
 			(effects
 				(font
@@
 		)
 		(property "Footprint" ""
-			(at 76.2 109.22 0)
+			(at 77.47 109.22 0)
 			(effects
 				(font
@@
 		)
 		(property "Datasheet" ""
-			(at 76.2 109.22 0)
+			(at 77.47 109.22 0)
 			(effects
 				(font
@@
 		)
 		(property "Description" "Power symbol creates a global label with name \"+3V3\""
-			(at 76.2 109.22 0)
+			(at 77.47 109.22 0)
 			(effects
 				(font
@@
 	)
 	(symbol
-		(lib_id "Device:L")
-		(at 205.74 52.07 90)
-		(unit 1)
-		(exclude_from_sim no)
-		(in_bom yes)
-		(on_board yes)
-		(dnp no)
-		(fields_autoplaced yes)
-		(property "Reference" "L1"
-			(at 205.74 46.99 90)
-			(effects
-				(font
-					(size 1.27 1.27)
-				)
-			)
-		)
-		(property "Value" "2nH"
-			(at 205.74 49.53 90)
-			(effects
-				(font
-					(size 1.27 1.27)
-				)
-			)
-		)
-		(property "Footprint" "Inductor_SMD:L_6.3x6.3_H3"
-			(at 205.74 52.07 0)
-			(effects
-				(font
-					(size 1.27 1.27)
-				)
-				(hide yes)
-			)
-		)
-		(property "Datasheet" "~"
-			(at 205.74 52.07 0)
-			(effects
-				(font
-					(size 1.27 1.27)
-				)
-				(hide yes)
-			)
-		)
-		(property "Description" "Inductor"
-			(at 205.74 52.07 0)
-			(effects
-				(font
-					(size 1.27 1.27)
-				)
-				(hide yes)
-			)
-		)
-		(pin "2"
-		)
-		(pin "1"
-		)
-		(instances
-			(project ""
-				(path "/6663287f-38c5-4c19-8add-d68d3434afcd"
-					(reference "L1")
-					(unit 1)
-				)
-			)
-		)
-	)
-	(symbol
 		(lib_id "power:VBUS")
 		(at 91.44 102.87 270)
@@
 			)
 		)
-		(property "Footprint" "Connector_PinSocket_2.54mm:PinSocket_1x04_P2.54mm_Horizontal"
+		(property "Footprint" "Connector_PinSocket_2.54mm:PinSocket_1x04_P2.54mm_Vertical"
 			(at 33.02 95.25 0)
 			(effects
@@
 			)
 		)
-		(property "Footprint" "Connector_PinSocket_2.54mm:PinSocket_1x04_P2.54mm_Horizontal"
+		(property "Footprint" "Connector_PinSocket_2.54mm:PinSocket_1x04_P2.54mm_Vertical"
 			(at 102.87 118.11 0)
 			(effects
@@
 	)
 	(symbol
+		(lib_id "Diode:1N4148WT")
+		(at 72.39 109.22 180)
+		(unit 1)
+		(exclude_from_sim no)
+		(in_bom yes)
+		(on_board yes)
+		(dnp no)
+		(fields_autoplaced yes)
+		(property "Reference" "D3"
+			(at 72.39 102.87 0)
+			(effects
+				(font
+					(size 1.27 1.27)
+				)
+			)
+		)
+		(property "Value" "1N4148WT"
+			(at 72.39 105.41 0)
+			(effects
+				(font
+					(size 1.27 1.27)
+				)
+			)
+		)
+		(property "Footprint" "Diode_SMD:D_SOD-523"
+			(at 72.39 104.775 0)
+			(effects
+				(font
+					(size 1.27 1.27)
+				)
+				(hide yes)
+			)
+		)
+		(property "Datasheet" "https://www.diodes.com/assets/Datasheets/ds30396.pdf"
+			(at 72.39 109.22 0)
+			(effects
+				(font
+					(size 1.27 1.27)
+				)
+				(hide yes)
+			)
+		)
+		(property "Description" "75V 0.15A Fast switching Diode, SOD-523"
+			(at 72.39 109.22 0)
+			(effects
+				(font
+					(size 1.27 1.27)
+				)
+				(hide yes)
+			)
+		)
+		(property "Sim.Device" "D"
+			(at 72.39 109.22 0)
+			(effects
+				(font
+					(size 1.27 1.27)
+				)
+				(hide yes)
+			)
+		)
+		(property "Sim.Pins" "1=K 2=A"
+			(at 72.39 109.22 0)
+			(effects
+				(font
+					(size 1.27 1.27)
+				)
+				(hide yes)
+			)
+		)
+		(pin "2"
+		)
+		(pin "1"
+		)
+		(instances
+			(project "Untitled"
+				(path "/6663287f-38c5-4c19-8add-d68d3434afcd"
+					(reference "D3")
+					(unit 1)
+				)
+			)
+		)
+	)
+	(symbol
 		(lib_id "Device:C")
 		(at 200.66 55.88 180)
@@
 					(unit 1)
 				)
-			)
-		)
-	)
-	(symbol
-		(lib_id "Device:D")
-		(at 55.88 149.86 180)
-		(unit 1)
-		(exclude_from_sim no)
-		(in_bom yes)
-		(on_board yes)
-		(dnp no)
-		(fields_autoplaced yes)
-		(property "Reference" "D2"
-			(at 55.88 143.51 0)
-			(effects
-				(font
-					(size 1.27 1.27)
-				)
-			)
-		)
-		(property "Value" "D"
-			(at 55.88 146.05 0)
-			(effects
-				(font
-					(size 1.27 1.27)
-				)
-			)
-		)
-		(property "Footprint" "Diode_SMD:D_0201_0603Metric"
-			(at 55.88 149.86 0)
-			(effects
-				(font
-					(size 1.27 1.27)
-				)
-				(hide yes)
-			)
-		)
-		(property "Datasheet" "~"
-			(at 55.88 149.86 0)
-			(effects
-				(font
-					(size 1.27 1.27)
-				)
-				(hide yes)
-			)
-		)
-		(property "Description" "Diode"
-			(at 55.88 149.86 0)
-			(effects
-				(font
-					(size 1.27 1.27)
-				)
-				(hide yes)
-			)
-		)
-		(property "Sim.Device" "D"
-			(at 55.88 149.86 0)
-			(effects
-				(font
-					(size 1.27 1.27)
-				)
-				(hide yes)
-			)
-		)
-		(property "Sim.Pins" "1=K 2=A"
-			(at 55.88 149.86 0)
-			(effects
-				(font
-					(size 1.27 1.27)
-				)
-				(hide yes)
-			)
-		)
-		(pin "1"
-		)
-		(pin "2"
-		)
-		(instances
-			(project ""
-				(path "/6663287f-38c5-4c19-8add-d68d3434afcd"
-					(reference "D2")
-					(unit 1)
-				)
