File: Kicad/Untitled/Untitled.kicad_sch (KiCad schematic)
At the start: 53 parts, among them J1 USB_C_Receptacle_USB2.0_14P, J2 Conn_01x04_Socket, J3 Screw_Terminal_01x02, J4 Conn_01x16_Pin, J5 Conn_01x04_Socket, J6 Conn_01x13_Pin, SW1 SW_Push_45deg, SW2 SW_Push_45deg, SW3 SW_Push, SW4 SW_Push, U1 NCP1117-3.3_TO252, U2 NCP1117-3.3_TO252, U3 APS6404L-3SQRx-ZR, U4 ESP32-S3, Y1 32.768kHz, Y2 40 MHz

Commit message: pcb update
Parts:
- removed D2, D3: 1N4148WT, Diode_SMD:D_SOD-523, symbol Diode:1N4148WT
- added D2, D3: D, Diode_SMD:D_0201_0603Metric, symbol Device:D
- J2, J5: footprint Connector_PinSocket_2.54mm:PinSocket_1x04_P2.54mm_Vertical -> Connector_PinSocket_2.54mm:PinSocket_1x04_P2.54mm_Horizontal
Connections:
- net +3V3: now also D3.1 (K)
- net VBUS: now also D2.2 (A); no longer C2.1, U2.3 (VI)
- net at C4.1, U2.2 (VO): now also D3.2 (A)
- new net: C2.1, D2.1 (K), U2.3 (VI)
Changed lines of the file:
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@@
 	)
 	(junction
-		(at 76.2 109.22)
-		(diameter 0)
-		(color 0 0 0 0)
-	)
-	(junction
 		(at 212.09 52.07)
 		(diameter 0)
@@
 	(wire
 		(pts
-			(xy 77.47 109.22) (xy 76.2 109.22)
+			(xy 85.09 149.86) (xy 83.82 149.86)
 		)
 		(stroke
@@
 	(wire
 		(pts
-			(xy 49.53 149.86) (xy 66.04 149.86)
+			(xy 49.53 149.86) (xy 52.07 149.86)
 		)
 		(stroke
@@
 	(wire
 		(pts
-			(xy 85.09 149.86) (xy 83.82 149.86)
-		)
-		(stroke
-			(width 0)
-			(type default)
-		)
-	)
-	(wire
-		(pts
 			(xy 207.01 142.24) (xy 208.28 142.24)
 		)
@@
 	(wire
 		(pts
+			(xy 59.69 149.86) (xy 66.04 149.86)
+		)
+		(stroke
+			(width 0)
+			(type default)
+		)
+	)
+	(wire
+		(pts
 			(xy 280.67 144.78) (xy 274.32 144.78)
 		)
@@
 	)
 	(symbol
-		(lib_id "Diode:1N4148WT")
-		(at 88.9 149.86 180)
-		(unit 1)
-		(exclude_from_sim no)
-		(in_bom yes)
-		(on_board yes)
-		(dnp no)
-		(fields_autoplaced yes)
-		(property "Reference" "D2"
-			(at 88.9 143.51 0)
-			(effects
-				(font
-					(size 1.27 1.27)
-				)
-			)
-		)
-		(property "Value" "1N4148WT"
-			(at 88.9 146.05 0)
-			(effects
-				(font
-					(size 1.27 1.27)
-				)
-			)
-		)
-		(property "Footprint" "Diode_SMD:D_SOD-523"
-			(at 88.9 145.415 0)
-			(effects
-				(font
-					(size 1.27 1.27)
-				)
-				(hide yes)
-			)
-		)
-		(property "Datasheet" "https://www.diodes.com/assets/Datasheets/ds30396.pdf"
-			(at 88.9 149.86 0)
-			(effects
-				(font
-					(size 1.27 1.27)
-				)
-				(hide yes)
-			)
-		)
-		(property "Description" "75V 0.15A Fast switching Diode, SOD-523"
-			(at 88.9 149.86 0)
-			(effects
-				(font
-					(size 1.27 1.27)
-				)
-				(hide yes)
-			)
-		)
-		(property "Sim.Device" "D"
-			(at 88.9 149.86 0)
-			(effects
-				(font
-					(size 1.27 1.27)
-				)
-				(hide yes)
-			)
-		)
-		(property "Sim.Pins" "1=K 2=A"
-			(at 88.9 149.86 0)
-			(effects
-				(font
-					(size 1.27 1.27)
-				)
-				(hide yes)
-			)
-		)
-		(pin "2"
-		)
-		(pin "1"
-		)
-		(instances
-			(project ""
-				(path "/6663287f-38c5-4c19-8add-d68d3434afcd"
-					(reference "D2")
-					(unit 1)
-				)
-			)
-		)
-	)
-	(symbol
 		(lib_id "Connector:Conn_01x16_Pin")
 		(at 83.82 85.09 0)
@@
 	)
 	(symbol
+		(lib_id "Device:D")
+		(at 88.9 149.86 180)
+		(unit 1)
+		(exclude_from_sim no)
+		(in_bom yes)
+		(on_board yes)
+		(dnp no)
+		(fields_autoplaced yes)
+		(property "Reference" "D3"
+			(at 88.9 143.51 0)
+			(effects
+				(font
+					(size 1.27 1.27)
+				)
+			)
+		)
+		(property "Value" "D"
+			(at 88.9 146.05 0)
+			(effects
+				(font
+					(size 1.27 1.27)
+				)
+			)
+		)
+		(property "Footprint" "Diode_SMD:D_0201_0603Metric"
+			(at 88.9 149.86 0)
+			(effects
+				(font
+					(size 1.27 1.27)
+				)
+				(hide yes)
+			)
+		)
+		(property "Datasheet" "~"
+			(at 88.9 149.86 0)
+			(effects
+				(font
+					(size 1.27 1.27)
+				)
+				(hide yes)
+			)
+		)
+		(property "Description" "Diode"
+			(at 88.9 149.86 0)
+			(effects
+				(font
+					(size 1.27 1.27)
+				)
+				(hide yes)
+			)
+		)
+		(property "Sim.Device" "D"
+			(at 88.9 149.86 0)
+			(effects
+				(font
+					(size 1.27 1.27)
+				)
+				(hide yes)
+			)
+		)
+		(property "Sim.Pins" "1=K 2=A"
+			(at 88.9 149.86 0)
+			(effects
+				(font
+					(size 1.27 1.27)
+				)
+				(hide yes)
+			)
+		)
+		(pin "1"
+		)
+		(pin "2"
+		)
+		(instances
+			(project "Untitled"
+				(path "/6663287f-38c5-4c19-8add-d68d3434afcd"
+					(reference "D3")
+					(unit 1)
+				)
+			)
+		)
+	)
+	(symbol
 		(lib_id "Regulator_Linear:NCP1117-3.3_TO252")
 		(at 59.69 109.22 0)
@@
 	(symbol
 		(lib_id "power:+3V3")
-		(at 77.47 109.22 0)
+		(at 76.2 109.22 0)
 		(unit 1)
 		(exclude_from_sim no)
@@
 		(fields_autoplaced yes)
 		(property "Reference" "#PWR09"
-			(at 77.47 113.03 0)
+			(at 76.2 113.03 0)
 			(effects
 				(font
@@
 		)
 		(property "Value" "+3V3"
-			(at 77.47 104.14 0)
+			(at 76.2 104.14 0)
 			(effects
 				(font
@@
 		)
 		(property "Footprint" ""
-			(at 77.47 109.22 0)
+			(at 76.2 109.22 0)
 			(effects
 				(font
@@
 		)
 		(property "Datasheet" ""
-			(at 77.47 109.22 0)
+			(at 76.2 109.22 0)
 			(effects
 				(font
@@
 		)
 		(property "Description" "Power symbol creates a global label with name \"+3V3\""
-			(at 77.47 109.22 0)
+			(at 76.2 109.22 0)
 			(effects
 				(font
@@
 			)
 		)
-		(property "Footprint" "Connector_PinSocket_2.54mm:PinSocket_1x04_P2.54mm_Vertical"
+		(property "Footprint" "Connector_PinSocket_2.54mm:PinSocket_1x04_P2.54mm_Horizontal"
 			(at 33.02 95.25 0)
 			(effects
@@
 			)
 		)
-		(property "Footprint" "Connector_PinSocket_2.54mm:PinSocket_1x04_P2.54mm_Vertical"
+		(property "Footprint" "Connector_PinSocket_2.54mm:PinSocket_1x04_P2.54mm_Horizontal"
 			(at 102.87 118.11 0)
 			(effects
@@
 	)
 	(symbol
-		(lib_id "Diode:1N4148WT")
-		(at 72.39 109.22 180)
-		(unit 1)
-		(exclude_from_sim no)
-		(in_bom yes)
-		(on_board yes)
-		(dnp no)
-		(fields_autoplaced yes)
-		(property "Reference" "D3"
-			(at 72.39 102.87 0)
-			(effects
-				(font
-					(size 1.27 1.27)
-				)
-			)
-		)
-		(property "Value" "1N4148WT"
-			(at 72.39 105.41 0)
-			(effects
-				(font
-					(size 1.27 1.27)
-				)
-			)
-		)
-		(property "Footprint" "Diode_SMD:D_SOD-523"
-			(at 72.39 104.775 0)
-			(effects
-				(font
-					(size 1.27 1.27)
-				)
-				(hide yes)
-			)
-		)
-		(property "Datasheet" "https://www.diodes.com/assets/Datasheets/ds30396.pdf"
-			(at 72.39 109.22 0)
-			(effects
-				(font
-					(size 1.27 1.27)
-				)
-				(hide yes)
-			)
-		)
-		(property "Description" "75V 0.15A Fast switching Diode, SOD-523"
-			(at 72.39 109.22 0)
-			(effects
-				(font
-					(size 1.27 1.27)
-				)
-				(hide yes)
-			)
-		)
-		(property "Sim.Device" "D"
-			(at 72.39 109.22 0)
-			(effects
-				(font
-					(size 1.27 1.27)
-				)
-				(hide yes)
-			)
-		)
-		(property "Sim.Pins" "1=K 2=A"
-			(at 72.39 109.22 0)
-			(effects
-				(font
-					(size 1.27 1.27)
-				)
-				(hide yes)
-			)
-		)
-		(pin "2"
-		)
-		(pin "1"
-		)
-		(instances
-			(project "Untitled"
-				(path "/6663287f-38c5-4c19-8add-d68d3434afcd"
-					(reference "D3")
-					(unit 1)
-				)
-			)
-		)
-	)
-	(symbol
 		(lib_id "Device:C")
 		(at 200.66 55.88 180)
@@
 					(unit 1)
 				)
+			)
+		)
+	)
+	(symbol
+		(lib_id "Device:D")
+		(at 55.88 149.86 180)
+		(unit 1)
+		(exclude_from_sim no)
+		(in_bom yes)
+		(on_board yes)
+		(dnp no)
+		(fields_autoplaced yes)
+		(property "Reference" "D2"
+			(at 55.88 143.51 0)
+			(effects
+				(font
+					(size 1.27 1.27)
+				)
+			)
+		)
+		(property "Value" "D"
+			(at 55.88 146.05 0)
+			(effects
+				(font
+					(size 1.27 1.27)
+				)
+			)
+		)
+		(property "Footprint" "Diode_SMD:D_0201_0603Metric"
+			(at 55.88 149.86 0)
+			(effects
+				(font
+					(size 1.27 1.27)
+				)
+				(hide yes)
+			)
+		)
+		(property "Datasheet" "~"
+			(at 55.88 149.86 0)
+			(effects
+				(font
+					(size 1.27 1.27)
+				)
+				(hide yes)
+			)
+		)
+		(property "Description" "Diode"
+			(at 55.88 149.86 0)
+			(effects
+				(font
+					(size 1.27 1.27)
+				)
+				(hide yes)
+			)
+		)
+		(property "Sim.Device" "D"
+			(at 55.88 149.86 0)
+			(effects
+				(font
+					(size 1.27 1.27)
+				)
+				(hide yes)
+			)
+		)
+		(property "Sim.Pins" "1=K 2=A"
+			(at 55.88 149.86 0)
+			(effects
+				(font
+					(size 1.27 1.27)
+				)
+				(hide yes)
+			)
+		)
+		(pin "1"
+		)
+		(pin "2"
+		)
+		(instances
+			(project ""
+				(path "/6663287f-38c5-4c19-8add-d68d3434afcd"
+					(reference "D2")
+					(unit 1)
+				)

Commit message: journal update, pcb update
Parts:
- removed C7, C8: 12pF, Capacitor_SMD:C_0402_1005Metric, symbol Device:C
- removed R4: 200, Resistor_SMD:R_0201_0603Metric, symbol Device:R
- removed U1, U2: NCP1117-3.3_TO252, Package_TO_SOT_SMD:TO-252-2, symbol Regulator_Linear:NCP1117-3.3_TO252
- removed Y1: 32.768kHz, AB38T_32_768KHZ:XTAL_AB38T-32.768KHZ, symbol Device:Crystal
- added U2, U6: LD1117S33TR_SOT223, Package_TO_SOT_SMD:SOT-223-3_TabPin2, symbol Regulator_Linear:LD1117S33TR_SOT223
- C1, C10, C11, C2, C3, C4: footprint Capacitor_SMD:C_0201_0603Metric -> Capacitor_SMD:C_0402_1005Metric
- D2, D3: footprint Diode_SMD:D_0201_0603Metric -> Diode_SMD:D_0402_1005Metric
- J1: footprint Connector_USB:USB_C_Receptacle_Amphenol_124019772112A -> TYPE-C-31-M-12:HRO_TYPE-C-31-M-12
- J3: footprint TerminalBlock:TerminalBlock_Altech_AK300-2_P5.00mm -> TerminalBlock_Phoenix:TerminalBlock_Phoenix_MKDS-1,5-2-5.08_1x02_P5.08mm_Horizontal
- R1, R14, R2, R3, R5, R6, R7, R8: footprint Resistor_SMD:R_0201_0603Metric -> Resistor_SMD:R_0402_1005Metric
- SW1, SW2, SW3, SW4: footprint Button_Switch_SMD:SW_Push_SPST_NO_Alps_SKRK -> Button_Switch_SMD:SW_SPST_B3U-1000P
Connections:
- net +3V3: now also D2.1 (K); no longer C3.1
- net GND: now also U2.1 (GND), U6.1 (GND)
- net VBUS: now also C2.1, U6.3 (VI); no longer D2.2 (A)
- net at C4.1, D3.2 (A): now also U6.2 (VO)
- net at C1.1, J3.1 (Pin_1): now also U2.3 (VI)
- net XTAL_32K_N: no longer names the net of U4.22 (XTAL_32K_N)
- net XTAL_32K_P: no longer names the net of U4.21 (XTAL_32K_P)
- new net: C3.1, D2.2 (A), U2.2 (VO)
- no-connect marks 4 -> 6
Other:
- moved on the sheet: C5, C6, R5, Y2
